File: encoder.kicad_sch (KiCad schematic)
At the start: 2 parts, among them IC1 AS5047P-ATSM

Commit message: Initial layout
Parts:
- C1: footprint (none) -> Capacitor_SMD:C_0603_1608Metric
Changed lines of the file:
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@@
 			)
 		)
-		(property "Footprint" ""
+		(property "Footprint" "Capacitor_SMD:C_0603_1608Metric"
 			(at 85.09 69.85 0)
 			(effects
