File: BLDC_Motor_Driver.kicad_pcb (KiCad board)
At the start: 2 copper layers, 135 x 111 mm, 95 parts, among them IC1 AS5047P-ATSM, IC10 INA214AIDCKT, IC12 INA214AIDCKT, IC13 INA214AIDCKT, IC2 L6498D, IC3 ATSAMD21G18A-MFT, IC5 ISL21090BFB812Z-TK, IC6 L6498D, IC7 L6498D, IC8 TPS7A4901DGNT, J1 FTSH-105-01-L-DV-K, J2 031-5431-10RFX, J3 031-5431-10RFX, J4 112405-12, J5 Conn_01x05_Pin, J6 Conn_01x04_Socket, J7 112405-12, J8 031-5431-10RFX, J9 Conn_01x03_Pin, Q1 IPB320N20N3GATMA1, Q2 IPB320N20N3GATMA1, Q3 IPB320N20N3GATMA1, Q4 IPB320N20N3GATMA1, Q5 IPB320N20N3GATMA1, Q6 IPB320N20N3GATMA1

Commit message: Finalize design
Parts:
- removed the G*** at (83.6, 125.3)
- added C19: 0.1uF, Capacitor_SMD:C_0603_1608Metric, F.Cu at (110.0, 90.6)
- added C25: 22pF, Capacitor_SMD:C_0603_1608Metric, F.Cu at (122.8, 102.5)
- added C26: 22pF, Capacitor_SMD:C_0603_1608Metric, F.Cu at (120.3, 100.2)
- added G***: LOGO, BLDC-Motor-Driver:kicad_logo, F.Cu at (146.1, 138.4)
- added G***: LOGO, BLDC-Motor-Driver:Bear, F.Cu at (94.9, 134.0)
- added IC4: TPL5010DDCT, BLDC-Motor-Driver:TPL5010DDCT, F.Cu at (110.4, 93.1)
- added R20: 20kΩ,1%, Resistor_SMD:R_0603_1608Metric, F.Cu at (106.7, 94.2)
- added Y1: ABS06-32.768KHZ-1-T, BLDC-Motor-Driver:ABS06, F.Cu at (120.4, 103.0)
- H1, H2, H3, H4: footprint MountingHole:MountingHole_4.3mm_M4_DIN965_Pad_TopBottom -> MountingHole:MountingHole_3.2mm_M3_DIN965_Pad
- R19, R6: value 1kΩ -> 10kΩ
- moved J4 102.4 mm to (155.6, 47.4)
- moved FB1 1.50 mm to (125.0, 105.5), turned to 90 degrees
- moved C29 0.26 mm to (166.8, 54.2)
- moved H2 0.05 mm to (148.1, 54.3)
- moved H4 0.05 mm to (148.1, 115.9)
Connections:
- IC3 pad 1: /Microcontroller/SERCOM1_PAD0 -> /Microcontroller/XIN32
- IC3 pad 2: unconnected-(IC3-PA01-Pad2) -> /Microcontroller/XOUT32
- IC3 pad 27: unconnected-(IC3-PA18-Pad27) -> /Microcontroller/SERCOM3_PAD2
- IC3 pad 38: unconnected-(IC3-PB23-Pad38) -> /Microcontroller/EXT_WDT_WAKE
- IC3 pad 39: unconnected-(IC3-PA27-Pad39) -> /Microcontroller/EXT_WDT_DONE
- J4 pad 5: /Microcontroller/SERCOM1_PAD0 -> /Microcontroller/SERCOM3_PAD2
Routing:
- net /Microcontroller/SERCOM3_PAD2: track 0.00 -> 64.6 mm, vias 0 -> 4
- net /Microcontroller/SERCOM1_PAD0: track 45.3 -> 0.00 mm, vias 2 -> 0
- net /Microcontroller/EXT_WDT_WAKE: track 0.00 -> 11.4 mm
- net /Microcontroller/EXT_WDT_DONE: track 0.00 -> 11.2 mm
- net /Microcontroller/XOUT32: track 0.00 -> 6.30 mm
- net /Microcontroller/XIN32: track 0.00 -> 5.06 mm
- net GND: track 80.6 -> 85.7 mm, vias 418 -> 111
- net /Microcontroller/RESET: track 41.9 -> 45.5 mm
- net Net-(IC4-DELAY/M_RST): track 0.00 -> 1.69 mm
- net /Microcontroller/SWDIO: track 48.8 -> 47.3 mm
- net +3V3: track 304.6 -> 305.7 mm, vias 16 -> 14
- net /Microcontroller/SERCOM4_PAD0: track 40.2 -> 41.3 mm
- net /Microcontroller/VDDANA: track 5.02 -> 5.92 mm
- removed copper zone on F.Cu, net GND
Other:
- board text added: "12V"
- board text added: "2mm"
- board text added: "5V"
- board text added: "PHASE A"
- board text added: "PHASE B"
- board text added: "PHASE C"
- board text added: "SWD Connector"
- board text added: "USART SERCOM 3"
- board text added: "USART SERCOM 4"
- board text added: "VBUS 20V"
