File: mcu.kicad_sch (KiCad schematic)
At the start: 11 parts, among them IC3 ATSAMD21G18A-MFT, J1 FTSH-105-01-L-DV-K

Commit message: Finalize design
Parts:
- added C19: 0.1uF, Capacitor_SMD:C_0603_1608Metric, symbol Device:C_Small
- added C25, C26: 22pF, Capacitor_SMD:C_0603_1608Metric, symbol Device:C_Small
- added IC4: TPL5010DDCT, BLDC-Motor-Driver:TPL5010DDCT, symbol BLDC-Motor-Driver_v2:TPL5010DDCT
- added R20: 20kΩ,1%, Resistor_SMD:R_0603_1608Metric, symbol Device:R_Small_US
- added Y1: ABS06-32.768KHZ-1-T, BLDC-Motor-Driver:ABS06, symbol BLDC-Motor-Driver_v2:ABS06-32.768KHZ-1-T
- R19, R6: value 1kΩ -> 10kΩ
Connections:
- net +3V3: now also C19.1, IC4.1 (VDD)
- net GND: now also C19.2, C25.2, C26.2, IC4.2 (GND), R20.2
- net RESET: now also IC4.6 (RSTN)
- net XOUT32: now reaches IC3.2 (PA01)
- net XOUT32: now also C25.1, Y1.2
- net SERCOM3_PAD2: now reaches IC3.27 (PA18)
- net EXT_WDT_WAKE: now reaches IC3.38 (PB23)
- net EXT_WDT_WAKE: now also IC4.5 (WAKE)
- net EXT_WDT_DONE: now reaches IC3.39 (PA27)
- net EXT_WDT_DONE: now also IC4.4 (DONE)
- net SERCOM1_PAD0 renamed XIN32
- net XIN32: now also C26.1, Y1.1
- new net: IC4.3 (DELAY/M_RST), R20.1
- no-connect marks 21 -> 17
Other:
- moved on the sheet: R19, R6
